File: Microcontrolador/PreliminarPCB.kicad_sch (KiCad schematic)
At the start: 8 parts, among them J1 Conn_01x20_Female, J2 Conn_01x20_Female, J3 Conn_01x08_Pin, SW1 SW_Push, SW2 SW_Push, SW3 SW_Push, SW4 SW_Push, SW5 SW_Push

Commit message: Se incluye esquema del rp2040
Parts:
- removed J3: Conn_01x08_Pin, symbol Connector:Conn_01x08_Pin
- removed SW1, SW2, SW3, SW4, SW5: SW_Push, symbol Switch:SW_Push
- added C1, C2: 27p, Capacitor_SMD:C_0402_1005Metric, symbol Device:C
- added C10, C8: 1u, Capacitor_SMD:C_0402_1005Metric, symbol Device:C
- added C11, C12, C13, C14, C15, C16, C4, C6, C7, C9: 100n, Capacitor_SMD:C_0402_1005Metric, symbol Device:C
- added C17, C3, C5: 10u, Capacitor_SMD:C_0805_2012Metric, symbol Device:C
- added H1, H2, H3, H4: MountingHole, MountingHole:MountingHole_2.7mm_M2.5, symbol Mechanical:MountingHole
- added J4: Conn_01x02, Connector_PinHeader_2.54mm:PinHeader_1x02_P2.54mm_Vertical, symbol Connector_Generic:Conn_01x02
- added J5: USB_B_Micro, RP2040_minimal:USB_Micro-B_Amphenol_10103594-0001LF_Horizontal_modified, symbol RP2040_minimal-rescue:USB_B_Micro-Connector
- added J6: Conn_01x08_Pin, symbol Connector:Conn_01x08_Pin
- added R1, R3: 1k, Capacitor_SMD:C_0402_1005Metric, symbol Device:R
- added R2: DNF, Capacitor_SMD:C_0402_1005Metric, symbol Device:R
- added R4, R5: 27, Capacitor_SMD:C_0402_1005Metric, symbol Device:R
- added SW10, SW6, SW7, SW8, SW9: SW_Push, symbol Switch:SW_Push
- added U1: NCP1117-3.3_SOT223, Package_TO_SOT_SMD:SOT-223-3_TabPin2, symbol Regulator_Linear:NCP1117-3.3_SOT223
- added U2: W25Q128JVS, Package_SO:SOIC-8_5.23x5.23mm_P1.27mm, symbol RP2040_minimal-rescue:W25Q128JVS-Memory_Flash
- added U3: RP2040, RP2040_minimal:RP2040-QFN-56, symbol MCU_RaspberryPi_RP2040:RP2040
- added Y1: ABLS-12.000MHZ-B4-T, RP2040_minimal:Crystal_SMD_HC49-US, symbol Device:Crystal
Connections:
- net +3.3V: now also J6.1 (Pin_1), J6.8 (Pin_8), SW10.1, SW6.1, SW7.1, SW8.1, SW9.1
- net CLK: now also J6.4 (Pin_4), U3.13 (GPIO10)
- net CS: now also J6.5 (Pin_5), U3.16 (GPIO13)
- net DC: now also J6.6 (Pin_6), U3.28 (GPIO17)
- net FALLA: now also U3.5 (GPIO3)
- net GFCI_TEST: now also U3.4 (GPIO2)
- net GND: now also C1.2, C10.2, C11.2, C12.2, C13.2, C14.2, C15.2, C16.2, C17.2, C2.2, C3.2, C4.2, C5.2, C6.2, C7.2, C8.2, C9.2, J4.2 (Pin_2), J5.5 (GND), J5.6 (Shield), J6.2 (Pin_2), U1.1 (GND), U2.4 (GND), U3.19 (TESTEN), U3.57 (GND)
- net NTC_Analog: now also U3.38 (GPIO26_ADC0)
- net RST: now also J6.7 (Pin_7), U3.31 (GPIO20)
- net RX_01: now also U3.7 (GPIO5)
- net SDA: now also J6.3 (Pin_3), U3.14 (GPIO11)
- net SW1: now also SW6.2, U3.8 (GPIO6)
- net SW2: now also SW7.2, U3.9 (GPIO7)
- net SW3: now also SW8.2, U3.11 (GPIO8)
- net SW4: now also SW9.2, U3.12 (GPIO9)
- net SW5: now also SW10.2, U3.32 (GPIO21)
- net TX_01: now also U3.6 (GPIO4)
- new net: C2.1, R3.2, Y1.2
- new net: R5.2, U3.46 (USB_DM)
- new net: R4.2, U3.47 (USB_DP)
- new net +1V1: C6.1, C7.1, C8.1, U3.23 (DVDD), U3.45 (VREG_VOUT), U3.50 (DVDD)
- new net +3V3: C10.1, C11.1, C12.1, C13.1, C14.1, C15.1, C16.1, C17.1, C4.1, C5.1, C9.1, R2.1, U1.2 (VO), U2.8 (VCC), U3.1 (IOVDD), U3.10 (IOVDD), U3.22 (IOVDD), U3.33 (IOVDD), U3.42 (IOVDD), U3.43 (ADC_AVDD), U3.44 (VREG_IN), U3.48 (USB_VDD), U3.49 (IOVDD)
- new net GPIO0: U3.2 (GPIO0)
- new net GPIO1: U3.3 (GPIO1)
- new net GPIO12: U3.15 (GPIO12)
- new net GPIO14: U3.17 (GPIO14)
- new net GPIO15: U3.18 (GPIO15)
- new net GPIO16: U3.27 (GPIO16)
- new net GPIO18: U3.29 (GPIO18)
- new net GPIO19: U3.30 (GPIO19)
- new net GPIO22: U3.34 (GPIO22)
- new net GPIO23: U3.35 (GPIO23)
- new net GPIO24: U3.36 (GPIO24)
- new net GPIO25: U3.37 (GPIO25)
- new net GPIO27_ADC1: U3.39 (GPIO27_ADC1)
- new net GPIO28_ADC2: U3.40 (GPIO28_ADC2)
- new net GPIO29_ADC3: U3.41 (GPIO29_ADC3)
- new net QSPI_SCLK: U2.6 (CLK), U3.52 (QSPI_SCLK)
- new net QSPI_SD0: U2.5 (DI(IO0)), U3.53 (QSPI_SD0)
- new net QSPI_SD1: U2.2 (DO(IO1)), U3.55 (QSPI_SD1)
- new net QSPI_SD2: U2.3 (IO2), U3.54 (QSPI_SD2)
- new net QSPI_SD3: U2.7 (IO3), U3.51 (QSPI_SD3)
- new net QSPI_SS: R1.1, R2.2, U2.1 (~{CS}), U3.56 (QSPI_SS)
- new net RUN: U3.26 (RUN)
- new net SWCLK: U3.24 (SWCLK)
- new net SWD: U3.25 (SWD)
- new net USB_D+: J5.3 (D+), R4.1
- new net USB_D-: J5.2 (D-), R5.1
- new net VBUS: C3.1, J5.1 (VBUS), U1.3 (VI)
- new net XIN: C1.1, U3.20 (XIN), Y1.1
- new net XOUT: R3.1, U3.21 (XOUT)
- new net ~{USB_BOOT}: J4.1 (Pin_1), R1.2
- no-connect marks 0 -> 1
Other:
- note added: "Cristal"
- note added: "Make sure C10 is close to pin 44 of RP2040"
- note added: "Make sure C8 is close to pin 45 of RP2040"
- note added: "Make sure R3 and R4 are close to RP2040"
- note added: "Memoria Flash"
- note added: "Power"
- moved on the sheet: J1, J2
