File: Potencia/PWM.kicad_sch (KiCad schematic)
At the start: 0 parts

Commit message: Bloques_CircuitoPotencia_ControlPilot
Parts:
- added C?: PGB1010603, symbols-footprints:ESD_PGB1010603MR, symbol PGB1010603:PGB1010603
- added C? (x2): 0.1uF 25V, Capacitor_THT:CP_Radial_D4.0mm_P1.50mm, symbol Device:C
- added R?: 1k Tol1%, Resistor_THT:R_Axial_DIN0204_L3.6mm_D1.6mm_P5.08mm_Horizontal, symbol Device:R
- added R? (x3): 200k Tol1%, Resistor_THT:R_Axial_DIN0204_L3.6mm_D1.6mm_P5.08mm_Horizontal, symbol Device:R
- added R?: 56k Tol1%, Resistor_THT:R_Axial_DIN0204_L3.6mm_D1.6mm_P5.08mm_Horizontal, symbol Device:R
- added R?: 66.5k Tol1%, Resistor_THT:R_Axial_DIN0204_L3.6mm_D1.6mm_P5.08mm_Horizontal, symbol Device:R
- added U?: LM324N, symbols-footprints:DIP794W45P254L1969H508Q14, symbol LM324N:LM324N
Connections:
- new net: R?.1, U?.1 (1OUT)
- new net: R?.1, R?.2, U?.2 (1IN-)
- new net +12V: C?.1, U?.4 (VCC)
- new net +3.3V: R?.1, R?.1
- new net -12V: C?.1, U?.11 (GND)
- new net GND: C?.1, C?.2, C?.2, R?.2, R?.2
- new net Pilot_ADC: R?.1, R?.2, R?.2
- new net Pilot_OUT: C?.2, R?.1, R?.2
- new net Pilot_PWM: U?.3 (1IN+)
- no-connect marks 0 -> 9
