File: Potencia/PWM.kicad_sch (KiCad schematic)
At the start: 10 parts

Commit message: guardado
Parts:
- removed C?: PGB1010603, symbols-footprints:ESD_PGB1010603MR, symbol PGB1010603:PGB1010603
- added D1: 1N4148, Diode_THT:D_DO-35_SOD27_P7.62mm_Horizontal, symbol Diode:1N4148
- gave numbers to parts that had none: 9
Connections:
- net GND: now also D1.2 (A)
- net Pilot_OUT: now also D1.1 (K)
