File: Potencia/micro.kicad_sch (KiCad schematic)
At the start: 0 parts

Commit message: correción de algunas referencias
Parts:
- added J3: Conn_01x08_Pin, symbol Connector:Conn_01x08_Pin
- added SW1, SW2, SW3, SW4, SW5: SW_Push, symbol Switch:SW_Push
- added U1: SC0915, RP2040:RP2040_SC0915, symbol RP2040:SC0915
Connections:
- new net +3.3V: J3.1 (Pin_1), J3.8 (Pin_8), SW1.1, SW2.1, SW3.1, SW4.1, SW5.1
- new net +5V: U1.40 (VBUS)
- new net CLK: J3.4 (Pin_4), U1.14 (I2C1_SDA/SPI1_SCK/GP10)
- new net CS: J3.5 (Pin_5), U1.17 (UART0_RX/I2C0_SCL/SPI1_CSn/GP13)
- new net DC: J3.6 (Pin_6), U1.22 (UART0_RX/I2C0_SCL/SPI0_CSn/GP17)
- new net FALLA: U1.5 (I2C1_SCL/SPI0_TX/GP3)
- new net GFCI_TEST: U1.4 (I2C1_SDA/SPI0_SCK/GP2)
- new net GND: J3.2 (Pin_2), U1.13 (GND), U1.18 (GND), U1.23 (GND), U1.28 (GND), U1.3 (GND), U1.33 (AGND/GND), U1.38 (GND), U1.8 (GND), U1.C (GND), U1.D (GND), U1.D2 (GND), U1.TP1 (GND)
- new net NTC_Analog: U1.31 (I2C1_SDA/ADC0/GP26)
- new net Pilot_ADC: U1.32 (I2C1_SCL/ADC1/GP27)
- new net Pilot_PWM: U1.29 (GP22)
- new net RST: J3.7 (Pin_7), U1.26 (I2C0_SDA/GP20)
- new net RX_01: U1.7 (UART1_RX/I2C0_SCL/SPI0_CSn/GP5)
- new net SDA: J3.3 (Pin_3), U1.15 (I2C1_SCL/SPI1_TX/GP11)
- new net SW1: SW1.2, U1.9 (I2C1_SDA/SPI0_SCK/GP6)
- new net SW2: SW2.2, U1.10 (I2C1_SCL/SPI0_TX/GP7)
- new net SW3: SW3.2, U1.11 (UART1_TX/I2C0_SDA/SPI1_RX/GP8)
- new net SW4: SW4.2, U1.12 (UART1_RX/I2C0_SCL/SPI1_CSn/GP9)
- new net SW5: SW5.2, U1.27 (I2C0_SCL/GP21)
- new net TX_01: U1.6 (UART1_TX/I2C0_SDA/SPI0_RX/GP4)
- new net USB_D+: U1.TP3 (USB_DP)
- new net USB_D-: U1.TP2 (USB_DM)
- no-connect marks 0 -> 6
Other:
- note added: "Pines de Salida del gc9a01"
- note added: "Pines de salida del Raspberry pi pico. Con sus conexiones."
- note added: "Switch de interfaz de usuario (Selección)"
