File: Potencia/_autosave-micro.kicad_sch (KiCad schematic)
At the start: 14 parts, among them J2 Relay, J3 Conn_01x08_Pin, Q1 PN2222A, Q2 PN2222A, SW1 SW_Push, SW2 SW_Push, SW3 SW_Push, SW4 SW_Push, SW5 SW_Push, U1 SC0915

Commit message: se añade relé, se corrigen parámetros
Parts:
- renumbered D4 to D2, D5 to D3, J3 to J?, R2 to R7, R3 to R8, SW5 to SW?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
