File: Potencia/CircuitoPotencia.kicad_sch (KiCad schematic)
At the start: 0 parts

Commit message: guardado
Other:
- removed sheet Potencia_Borrador
- added sheet Sensores (Sensores.kicad_sch)
Changed lines of the file:
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@@
-    (effects (font (size 1.27 1.27)) (justify left bottom))
-  )
-  (text "Esta etapa aparece aislada porque\ntodas sus conexiones con los demás\nmódulos son variables globales y\npor eso no aparenta tener I/O"
-    (at 62.23 80.01 0)
     (effects (font (size 1.27 1.27)) (justify left bottom))
   )
@@
       (project "CircuitoPotencia"
         (path "/f64e4c48-29c2-4644-b6e3-d55b9152fc29" (page "4"))
+      )
+    )
+  )
+  (sheet (at 57.15 43.18) (size 46.99 35.56) (fields_autoplaced)
+    (stroke (width 0.1524) (type solid))
+    (fill (color 0 0 0 0.0000))
+    (property "Sheetname" "Sensores" (at 57.15 42.4684 0)
+      (effects (font (size 1.27 1.27)) (justify left bottom))
+    )
+    (property "Sheetfile" "Sensores.kicad_sch" (at 57.15 79.3246 0)
+      (effects (font (size 1.27 1.27)) (justify left top))
+    )
+    (instances
+      (project "CircuitoPotencia"
+        (path "/f64e4c48-29c2-4644-b6e3-d55b9152fc29" (page "6"))
       )
     )
@@
       )
     )
-  )
-  (sheet (at 59.69 41.91) (size 35.56 25.4) (fields_autoplaced)
-    (stroke (width 0.1524) (type solid))
-    (fill (color 0 0 0 0.0000))
-    (property "Sheetname" "Potencia_Borrador" (at 59.69 41.1984 0)
-      (effects (font (size 1.27 1.27)) (justify left bottom))
-    )
-    (property "Sheetfile" "Potencia.kicad_sch" (at 59.69 67.8946 0)
-      (effects (font (size 1.27 1.27)) (justify left top))
-    )
-    (instances
-      (project "CircuitoPotencia"
-        (path "/f64e4c48-29c2-4644-b6e3-d55b9152fc29" (page "2"))
-      )
-    )
