File: Potencia/untitled.kicad_sch (KiCad schematic)
At the start: 13 parts, among them U3.3 LM2596S-3.3, U5 LM2596S-5

Commit message: Bloques_CircuitoPotencia_ControlPilot
Other:
- moved on the sheet: CIn0, CIn2, COut1, COut2, Cin1, D1, D2, DIn, JP?, L1, L2, U3.3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

Commit message: Potencia_actualiza
Parts:
- added CIn?: 1u, symbol Device:C
- added CIn?: 2.2u, symbol Device:C
- added U?: LM7912_TO220, Package_TO_SOT_THT:TO-220-3_Vertical, symbol Regulator_Linear:LM7912_TO220
Connections:
- net GND: now also CIn?.1, CIn?.1, U?.1 (GND)
- new net: CIn?.2, U?.3 (VO)
- new net: CIn?.2, U?.2 (VI)
Changed lines of the file:
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@@
   (junction (at 201.93 63.5) (diameter 0) (color 0 0 0 0)
   )
+  (junction (at 100.33 160.02) (diameter 0) (color 0 0 0 0)
+  )
   (junction (at 223.52 63.5) (diameter 0) (color 0 0 0 0)
   )
@@
     (stroke (width 0) (type default) (color 0 0 0 0))
   )
+  (wire (pts (xy 68.58 147.32) (xy 100.33 147.32))
+    (stroke (width 0) (type default) (color 0 0 0 0))
+  )
   (wire (pts (xy 110.49 88.9) (xy 118.11 88.9))
     (stroke (width 0) (type default) (color 0 0 0 0))
@@
     (stroke (width 0) (type default) (color 0 0 0 0))
   )
+  (wire (pts (xy 100.33 160.02) (xy 114.3 160.02))
+    (stroke (width 0) (type default) (color 0 0 0 0))
+  )
   (wire (pts (xy 201.93 115.57) (xy 201.93 118.11))
     (stroke (width 0) (type default) (color 0 0 0 0))
@@
     (stroke (width 0) (type default) (color 0 0 0 0))
   )
+  (wire (pts (xy 107.95 176.53) (xy 114.3 176.53))
+    (stroke (width 0) (type default) (color 0 0 0 0))
+  )
   (wire (pts (xy 201.93 63.5) (xy 209.55 63.5))
     (stroke (width 0) (type default) (color 0 0 0 0))
@@
     (stroke (width 0) (type default) (color 0 0 0 0))
   )
+  (wire (pts (xy 83.82 176.53) (xy 92.71 176.53))
+    (stroke (width 0) (type default) (color 0 0 0 0))
+  )
+  (wire (pts (xy 100.33 160.02) (xy 100.33 168.91))
+    (stroke (width 0) (type default) (color 0 0 0 0))
+  )
   (wire (pts (xy 196.85 115.57) (xy 201.93 115.57))
     (stroke (width 0) (type default) (color 0 0 0 0))
   )
+  (wire (pts (xy 114.3 160.02) (xy 114.3 162.56))
+    (stroke (width 0) (type default) (color 0 0 0 0))
+  )
   (wire (pts (xy 147.32 58.42) (xy 154.94 58.42))
     (stroke (width 0) (type default) (color 0 0 0 0))
@@
     (stroke (width 0) (type default) (color 0 0 0 0))
   )
+  (wire (pts (xy 83.82 160.02) (xy 100.33 160.02))
+    (stroke (width 0) (type default) (color 0 0 0 0))
+  )
   (wire (pts (xy 168.91 115.57) (xy 168.91 128.27))
     (stroke (width 0) (type default) (color 0 0 0 0))
@@
     (stroke (width 0) (type default) (color 0 0 0 0))
   )
+  (wire (pts (xy 100.33 147.32) (xy 100.33 160.02))
+    (stroke (width 0) (type default) (color 0 0 0 0))
+  )
   (wire (pts (xy 196.85 63.5) (xy 201.93 63.5))
     (stroke (width 0) (type default) (color 0 0 0 0))
@@
     (stroke (width 0) (type default) (color 0 0 0 0))
   )
+  (wire (pts (xy 83.82 170.18) (xy 83.82 176.53))
+    (stroke (width 0) (type default) (color 0 0 0 0))
+  )
   (wire (pts (xy 223.52 73.66) (xy 223.52 76.2))
     (stroke (width 0) (type default) (color 0 0 0 0))
   )
+  (wire (pts (xy 83.82 162.56) (xy 83.82 160.02))
+    (stroke (width 0) (type default) (color 0 0 0 0))
+  )
   (polyline (pts (xy 33.02 69.85) (xy 125.73 69.85))
+    (stroke (width 0) (type default) (color 0 0 0 0))
+  )
+  (wire (pts (xy 114.3 176.53) (xy 114.3 170.18))
     (stroke (width 0) (type default) (color 0 0 0 0))
   )
@@
     (pin "2")
   )
+  (symbol (lib_id "Device:C") (at 114.3 166.37 0) (unit 1)
+    (in_bom yes) (on_board yes) (fields_autoplaced)
+    (property "Reference" "CIn?" (id 0) (at 118.11 165.0999 0)
+      (effects (font (size 1.27 1.27)) (justify left))
+    )
+    (property "Value" "1u" (id 1) (at 118.11 167.6399 0)
+      (effects (font (size 1.27 1.27)) (justify left))
+    )
+    (property "Footprint" "" (id 2) (at 115.2652 170.18 0)
+      (effects (font (size 1.27 1.27)) hide)
+    )
+    (property "Datasheet" "~" (id 3) (at 114.3 166.37 0)
+      (effects (font (size 1.27 1.27)) hide)
+    )
+    (pin "1")
+    (pin "2")
+  )
   (symbol (lib_id "power:GND") (at 154.94 76.2 0) (unit 1)
     (in_bom yes) (on_board yes) (fields_autoplaced)
@@
     )
     (pin "1")
+  )
+  (symbol (lib_id "Regulator_Linear:LM7912_TO220") (at 100.33 176.53 0) (unit 1)
+    (in_bom yes) (on_board yes) (fields_autoplaced)
+    (property "Reference" "U?" (id 0) (at 100.33 181.61 0))
+    (property "Value" "LM7912_TO220" (id 1) (at 100.33 184.15 0))
+    (property "Footprint" "Package_TO_SOT_THT:TO-220-3_Vertical" (id 2) (at 100.33 181.61 0)
+      (effects (font (size 1.27 1.27) italic) hide)
+    )
+    (property "Datasheet" "hhttps://www.onsemi.com/pub/Collateral/MC7900-D.PDF" (id 3) (at 100.33 176.53 0)
+      (effects (font (size 1.27 1.27)) hide)
+    )
+    (pin "1")
+    (pin "2")
+    (pin "3")
   )
   (symbol (lib_id "power:GND") (at 154.94 128.27 0) (unit 1)
@@
     (pin "2")
   )
+  (symbol (lib_id "Device:C") (at 83.82 166.37 0) (unit 1)
+    (in_bom yes) (on_board yes) (fields_autoplaced)
+    (property "Reference" "CIn?" (id 0) (at 87.63 165.0999 0)
+      (effects (font (size 1.27 1.27)) (justify left))
+    )
+    (property "Value" "2.2u" (id 1) (at 87.63 167.6399 0)
+      (effects (font (size 1.27 1.27)) (justify left))
+    )
+    (property "Footprint" "" (id 2) (at 84.7852 170.18 0)
+      (effects (font (size 1.27 1.27)) hide)
+    )
+    (property "Datasheet" "~" (id 3) (at 83.82 166.37 0)
+      (effects (font (size 1.27 1.27)) hide)
+    )
+    (pin "1")
+    (pin "2")
+  )
   (symbol (lib_id "power:+12V") (at 110.49 82.55 0) (unit 1)
     (in_bom yes) (on_board yes) (fields_autoplaced)
@@
       (effects (font (size 1.27 1.27)) hide)
     )
+    (pin "1")
+  )
+  (symbol (lib_id "power:GND") (at 68.58 147.32 0) (unit 1)
+    (in_bom yes) (on_board yes) (fields_autoplaced)
+    (property "Reference" "#PWR?" (id 0) (at 68.58 153.67 0)
+      (effects (font (size 1.27 1.27)) hide)
+    )
+    (property "Value" "GND" (id 1) (at 68.58 152.4 0))
+    (property "Footprint" "" (id 2) (at 68.58 147.32 0)
+      (effects (font (size 1.27 1.27)) hide)
+    )
+    (property "Datasheet" "" (id 3) (at 68.58 147.32 0)
+      (effects (font (size 1.27 1.27)) hide)
+    )

Commit message: Actualización de carpeta Control Pilot
Parts:
- CIn0: value 22uF -> (none); footprint Capacitor_SMD:C_0805_2012Metric_Pad1.18x1.45mm_HandSolder -> (none)
- CIn2, Cin1: value 680u -> (none)
- CIn?: value 1u -> (none)
- CIn?: value 2.2u -> (none)
- COut1, COut2: value 220u -> (none)
- D1, D2: value 1N5822 -> (none); footprint Diode_THT:D_DO-201AD_P15.24mm_Horizontal -> (none)
- DIn: value 1N4007 -> (none); footprint Diode_SMD:D_SMA_Handsoldering -> (none)
- JP?: value Jumper_3_Open -> (none); footprint Connector_PinHeader_2.54mm:PinHeader_1x03_P2.54mm_Vertical -> (none)
- L1, L2: value 33u -> (none)
- U3.3: value LM2596S-3.3 -> (none); footprint Package_TO_SOT_SMD:TO-263-5_TabPin3 -> (none)
- U5: value LM2596S-5 -> (none); footprint Package_TO_SOT_SMD:TO-263-5_TabPin3 -> (none)
- U?: value LM7912_TO220 -> (none); footprint Package_TO_SOT_THT:TO-220-3_Vertical -> (none)
Other:
- moved on the sheet: CIn?, U?
