File: Esquemático_UNCargador/untitled.kicad_sch (KiCad schematic)
At the start: 18 parts, among them U3.3 LM2596S-3.3, U5 LM2596S-5

Commit message: NuevaHuellaPot
Parts:
- added PS2: LM2596_3.3_ADJ, LM2596ADJ:LM2596ADJ, symbol Converter_DCDC:ITX0503SA-H
Other:
- moved on the sheet: LM2596ADJ_3.3
Changed lines of the file:
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@@
+    )
+  )
+  (symbol (lib_name "+12V_1") (lib_id "power:+12V") (at 47.3456 153.8478 0) (unit 1)
+    (in_bom yes) (on_board yes) (dnp no) (fields_autoplaced)
+    (property "Reference" "#PWR01" (at 47.3456 157.6578 0)
+      (effects (font (size 1.27 1.27)) hide)
+    )
+    (property "Value" "+12V" (at 47.3456 149.86 0)
+      (effects (font (size 1.27 1.27)))
+    )
+    (property "Footprint" "" (at 47.3456 153.8478 0)
+      (effects (font (size 1.27 1.27)) hide)
+    )
+    (property "Datasheet" "" (at 47.3456 153.8478 0)
+      (effects (font (size 1.27 1.27)) hide)
+    )
+    (pin "1")
+    (instances
+      (project "untitled"
+        (path "/9be105a0-504f-4b07-b004-211a0f61b6b4"
+          (reference "#PWR01") (unit 1)
+        )
+      )
     )
   )
@@
     )
   )
-  (symbol (lib_id "LM2596ADJ:LM2596ADJ") (at 40.5384 124.5362 0) (unit 1)
-    (in_bom yes) (on_board yes) (dnp no) (fields_autoplaced)
-    (property "Reference" "LM2596ADJ_3.3" (at 40.5384 125.73 0)
-      (effects (font (size 1.27 1.27)))
-    )
-    (property "Value" "ADJ3.3V" (at 40.5384 124.5362 0)
-      (effects (font (size 1.27 1.27)))
-    )
-    (property "Footprint" "LM2596ADJ:LM2596ADJ" (at 40.5384 124.5362 0)
-      (effects (font (size 1.27 1.27)) hide)
-    )
-    (property "Datasheet" "" (at 40.5384 124.5362 0)
+  (symbol (lib_id "LM2596ADJ:LM2596ADJ") (at 62.3062 150.241 0) (unit 1)
+    (in_bom yes) (on_board yes) (dnp no) (fields_autoplaced)
+    (property "Reference" "LM2596ADJ_3.3" (at 62.3062 151.4348 0)
+      (effects (font (size 1.27 1.27)))
+    )
+    (property "Value" "ADJ3.3V" (at 62.3062 150.241 0)
+      (effects (font (size 1.27 1.27)))
+    )
+    (property "Footprint" "LM2596ADJ:LM2596ADJ" (at 62.3062 150.241 0)
+      (effects (font (size 1.27 1.27)) hide)
+    )
+    (property "Datasheet" "" (at 62.3062 150.241 0)
       (effects (font (size 1.27 1.27)) hide)
     )
@@
         )
       )
+    )
+  )
+  (symbol (lib_id "Converter_DCDC:ITX0503SA-H") (at 51.3842 134.0358 0) (unit 1)
+    (in_bom yes) (on_board yes) (dnp no) (fields_autoplaced)
+    (property "Reference" "PS2" (at 51.3842 124.46 0)
+      (effects (font (size 1.27 1.27)))
+    )
+    (property "Value" "LM2596_3.3_ADJ" (at 51.3842 127 0)
+      (effects (font (size 1.27 1.27)))
+    )
+    (property "Footprint" "LM2596ADJ:LM2596ADJ" (at 24.7142 140.3858 0)
+      (effects (font (size 1.27 1.27)) (justify left) hide)
+    )
+    (property "Datasheet" "https://www.xppower.com/pdfs/SF_ITX.pdf" (at 78.0542 141.6558 0)
+      (effects (font (size 1.27 1.27)) (justify left) hide)
+    )
+    (pin "1")
+    (pin "2")
+    (pin "6")
+    (pin "7")
+    (pin "8")
+    (instances
+      (project "untitled"
+        (path "/9be105a0-504f-4b07-b004-211a0f61b6b4"
+          (reference "PS2") (unit 1)
+        )
+      )

Commit message: Cambios de recomendaciones profesor
Parts:
- removed DIn: 1N4007, Diode_SMD:D_SMA_Handsoldering, symbol Diode:1N4007
Connections:
- net +12V: now also CIn?.2, JP1.3 (B), U?.2 (VI)
- net N: now reaches PS1.1 (AC/N)
- net In110v: now reaches PS1.2 (AC/L)
Changed lines of the file:
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@@
   (junction (at 92.71 83.82) (diameter 0) (color 0 0 0 0)
   )
+  (junction (at 107.95 163.83) (diameter 0) (color 0 0 0 0)
+  )
   (junction (at 261.62 105.41) (diameter 0) (color 0 0 0 0)
   )
@@
     (stroke (width 0) (type default))
   )
+  (wire (pts (xy 107.95 163.83) (xy 93.98 163.83))
+    (stroke (width 0) (type default))
+  )
   (wire (pts (xy 148.59 78.74) (xy 156.21 78.74))
     (stroke (width 0) (type default))
@@
     (stroke (width 0) (type default))
   )
+  (wire (pts (xy 39.37 83.82) (xy 45.72 83.82))
+    (stroke (width 0) (type default))
+  )
   (wire (pts (xy 105.41 77.47) (xy 105.41 78.74))
     (stroke (width 0) (type default))
@@
     (stroke (width 0) (type default))
   )
+  (wire (pts (xy 39.37 78.74) (xy 45.72 78.74))
+    (stroke (width 0) (type default))
+  )
   (wire (pts (xy 261.62 43.18) (xy 261.62 48.26))
     (stroke (width 0) (type default))
@@
     (stroke (width 0) (type default))
   )
-  (wire (pts (xy 133.35 78.74) (xy 148.59 78.74))
-    (stroke (width 0) (type default))
-  )
   (wire (pts (xy 207.01 53.34) (xy 209.55 53.34))
     (stroke (width 0) (type default))
@@
     (stroke (width 0) (type default))
   )
+  (wire (pts (xy 93.98 163.83) (xy 93.98 161.29))
+    (stroke (width 0) (type default))
+  )
   (wire (pts (xy 261.62 115.57) (xy 261.62 118.11))
     (stroke (width 0) (type default))
@@
     (stroke (width 0) (type default))
   )
-  (wire (pts (xy 111.76 78.74) (xy 125.73 78.74))
+  (wire (pts (xy 111.76 78.74) (xy 148.59 78.74))
     (stroke (width 0) (type default))
   )
@@
     (effects (font (size 1.27 1.27)) (justify left bottom))
   )
+  (hierarchical_label "In110v" (shape input) (at 39.37 78.74 180) (fields_autoplaced)
+    (effects (font (size 1.27 1.27)) (justify right))
+  )
+  (hierarchical_label "N" (shape input) (at 39.37 83.82 180) (fields_autoplaced)
+    (effects (font (size 1.27 1.27)) (justify right))
+  )
   (symbol (lib_id "power:GND") (at 240.03 118.11 0) (unit 1)
     (in_bom yes) (on_board yes) (dnp no) (fields_autoplaced)
@@
         )
       )
+      (project "CircuitoPotencia"
+        (path "/f64e4c48-29c2-4644-b6e3-d55b9152fc29/c38372d7-094a-4ec0-82ac-c3a161d378bf"
+          (reference "#PWR0123") (unit 1)
+        )
+      )
     )
   )
@@
         )
       )
+      (project "CircuitoPotencia"
+        (path "/f64e4c48-29c2-4644-b6e3-d55b9152fc29/c38372d7-094a-4ec0-82ac-c3a161d378bf"
+          (reference "LM2596ADJ_3.3") (unit 1)
+        )
+      )
     )
   )
@@
         (path "/f64e4c48-29c2-4644-b6e3-d55b9152fc29/c38372d7-094a-4ec0-82ac-c3a161d378bf"
           (reference "U3") (unit 1)
+        )
+      )
+    )
+  )
+  (symbol (lib_id "power:+12V") (at 93.98 161.29 0) (unit 1)
+    (in_bom yes) (on_board yes) (dnp no)
+    (property "Reference" "#PWR0101" (at 93.98 165.1 0)
+      (effects (font (size 1.27 1.27)) hide)
+    )
+    (property "Value" "+12V" (at 93.98 157.48 0)
+      (effects (font (size 1.27 1.27)))
+    )
+    (property "Footprint" "" (at 93.98 161.29 0)
+      (effects (font (size 1.27 1.27)) hide)
+    )
+    (property "Datasheet" "" (at 93.98 161.29 0)
+      (effects (font (size 1.27 1.27)) hide)
+    )
+    (pin "1")
+    (instances
+      (project "untitled"
+        (path "/9be105a0-504f-4b07-b004-211a0f61b6b4"
+          (reference "#PWR0101") (unit 1)
+        )
+      )
+      (project "CircuitoPotencia"
+        (path "/f64e4c48-29c2-4644-b6e3-d55b9152fc29/758fec3f-d66e-4356-8861-1c58650d5bb5"
+          (reference "#PWR0101") (unit 1)
+        )
+        (path "/f64e4c48-29c2-4644-b6e3-d55b9152fc29/c38372d7-094a-4ec0-82ac-c3a161d378bf"
+          (reference "#PWR012") (unit 1)
         )
       )
@@
         )
       )
+      (project "CircuitoPotencia"
+        (path "/f64e4c48-29c2-4644-b6e3-d55b9152fc29/c38372d7-094a-4ec0-82ac-c3a161d378bf"
+          (reference "PS2") (unit 1)
+        )
+      )
     )
   )
@@
         )
       )
-    )
-  )
-  (symbol (lib_id "Diode:1N4007") (at 129.54 78.74 180) (unit 1)
-    (in_bom yes) (on_board yes) (dnp no) (fields_autoplaced)
-    (property "Reference" "DIn" (at 129.54 72.39 0)
-      (effects (font (size 1.27 1.27)))
-    )
-    (property "Value" "1N4007" (at 129.54 74.93 0)
-      (effects (font (size 1.27 1.27)))
-    )
-    (property "Footprint" "Diode_SMD:D_SMA_Handsoldering" (at 129.54 74.295 0)
-      (effects (font (size 1.27 1.27)) hide)
-    )
-    (property "Datasheet" "http://www.vishay.com/docs/88503/1n4001.pdf" (at 129.54 78.74 0)
-      (effects (font (size 1.27 1.27)) hide)
-    )
-    (pin "1")
-    (pin "2")
-    (instances
-      (project "untitled"
-        (path "/9be105a0-504f-4b07-b004-211a0f61b6b4"
-          (reference "DIn") (unit 1)
-        )
-      )
-      (project "CircuitoPotencia"
-        (path "/f64e4c48-29c2-4644-b6e3-d55b9152fc29/c38372d7-094a-4ec0-82ac-c3a161d378bf"
-          (reference "DIn1") (unit 1)
-        )
-      )
