File: Esquemático_UNCargador/micro.kicad_sch (KiCad schematic)
At the start: 19 parts, among them J1 Conn_01x04_Pin, J2 Relay1, J9 Relay2, Q1 PN2222A, Q2 PN2222A

Commit message: PCB con ruteo realizado. Errores en los anchos de vias -0.2mm. Huella LF356n actualizada
Connections:
- net DIsplaySCL is gone; now on net DisplaySCL: J1.4 (Pin_4)
Changed lines of the file:
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@@
-    )
-  )
-  (global_label "Pilot_PWM" (shape input) (at 139.7 73.66 0) (fields_autoplaced)
-    (effects (font (size 1.27 1.27)) (justify left))
-    (property "Intersheetrefs" "${INTERSHEET_REFS}" (at 152.1609 73.66 0)
-      (effects (font (size 1.27 1.27)) (justify left) hide)
     )
   )
@@
     )
   )
-  (global_label "DIsplaySCL" (shape bidirectional) (at 130.81 171.45 0) (fields_autoplaced)
+  (global_label "DisplaySCL" (shape bidirectional) (at 130.81 171.45 0) (fields_autoplaced)
     (effects (font (size 1.27 1.27)) (justify left))
     (property "Intersheetrefs" "${INTERSHEET_REFS}" (at 145.1684 171.45 0)
@@
     (effects (font (size 1.27 1.27)) (justify left))
   )
+  (hierarchical_label "Pilot_PWM" (shape input) (at 139.7 73.66 0) (fields_autoplaced)
+    (effects (font (size 1.27 1.27)) (justify left))
+  )
