File: Esquemático_UNCargador/CircuitoPotencia.kicad_sch (KiCad schematic)
At the start: 2 parts, among them J2 Neutro, J3 Conn_02x03_Counter_Clockwise

Commit message: PCB_Final
Parts:
- J3: footprint Connector_IDC:IDC-Header_2x04_P2.54mm_Vertical -> Connector_IDC:IDC-Header_2x05_P2.54mm_Vertical
Changed lines of the file:
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@@
       (effects (font (size 1.27 1.27)) (justify right))
     )
-    (property "Footprint" "Connector_IDC:IDC-Header_2x04_P2.54mm_Vertical" (at 22.86 137.16 0)
+    (property "Footprint" "Connector_IDC:IDC-Header_2x05_P2.54mm_Vertical" (at 22.86 137.16 0)
       (effects (font (size 1.27 1.27)) hide)
     )
