File: Esquemático_UNCargador/CircuitoPotencia.kicad_pcb (KiCad board)
At the start: 2 copper layers, 143.9 x 141 mm, 61 parts, among them IC1 LF353, J1 Conn_01x04_Pin, J2 Relay1, J3 Conn_02x03_Counter_Clockwise, J4 GFCI, J5 PZEM 004T 100A, J6 NTC 3950, J8 Conn_01x02_Pin, J9 Relay2, Q1 PN2222A, Q2 PN2222A, SW1 SW_Push, SW2 SW_Push, SW3 SW_Push, SW4 SW_Push, SW5 SW_Push, U2 LF356, U3 LM7912(Inversor)

Commit message: Cambio huella J3 embebidos
Parts:
- J3: footprint Connector_PinHeader_2.54mm:PinHeader_2x03_P2.54mm_Vertical -> Connector_IDC:IDC-Header_2x04_P2.54mm_Vertical
Routing:
- net /Microcontrolador/SPI0_TX: track 18.4 -> 22.1 mm
Changed lines of the file:
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@@
     )
   )
-  (footprint "Connector_PinHeader_2.54mm:PinHeader_2x03_P2.54mm_Vertical" (layer "F.Cu")
+  (footprint "Connector_IDC:IDC-Header_2x04_P2.54mm_Vertical" (layer "F.Cu")
     (at 49.53 99.06)
-    (descr "Through hole straight pin header, 2x03, 2.54mm pitch, double rows")
-    (tags "Through hole pin header THT 2x03 2.54mm double row")
+    (descr "Through hole IDC box header, 2x04, 2.54mm pitch, DIN 41651 / IEC 60603-13, double rows, https://docs.google.com/spreadsheets/d/16SsEcesNF15N3Lb4niX7dcUr-NY5_MFPQhobNuNppn4/edit#gid=0")
+    (tags "Through hole vertical IDC box header THT 2x04 2.54mm double row")
     (property "Sheetfile" "CircuitoPotencia.kicad_sch")
     (property "Sheetname" "")
@@
     (property "ki_keywords" "connector")
     (attr through_hole)
-    (fp_text reference "J3" (at 1.27 -2.33) (layer "F.SilkS")
+    (fp_text reference "J3" (at 1.27 -6.1) (layer "F.SilkS")
         (effects (font (size 1 1) (thickness 0.15)))
     )
-    (fp_text value "Conn_02x03_Counter_Clockwise" (at 1.27 7.41) (layer "F.Fab")
+    (fp_text value "Conn_02x03_Counter_Clockwise" (at 1.27 13.72) (layer "F.Fab")
         (effects (font (size 1 1) (thickness 0.15)))
     )
-    (fp_text user "${REFERENCE}" (at 1.27 2.54 90) (layer "F.Fab")
+    (fp_text user "${REFERENCE}" (at 1.27 3.81 90) (layer "F.Fab")
         (effects (font (size 1 1) (thickness 0.15)))
     )
-    (fp_line (start -1.33 -1.33) (end 0 -1.33)
+    (fp_line (start -4.68 -0.5) (end -4.68 0.5)
       (stroke (width 0.12) (type solid)) (layer "F.SilkS"))
-    (fp_line (start -1.33 0) (end -1.33 -1.33)
+    (fp_line (start -4.68 0.5) (end -3.68 0)
       (stroke (width 0.12) (type solid)) (layer "F.SilkS"))
-    (fp_line (start -1.33 1.27) (end -1.33 6.41)
+    (fp_line (start -3.68 0) (end -4.68 -0.5)
       (stroke (width 0.12) (type solid)) (layer "F.SilkS"))
-    (fp_line (start -1.33 1.27) (end 1.27 1.27)
+    (fp_line (start -3.29 -5.21) (end 5.83 -5.21)
       (stroke (width 0.12) (type solid)) (layer "F.SilkS"))
-    (fp_line (start -1.33 6.41) (end 3.87 6.41)
+    (fp_line (start -3.29 1.76) (end -1.98 1.76)
       (stroke (width 0.12) (type solid)) (layer "F.SilkS"))
-    (fp_line (start 1.27 -1.33) (end 3.87 -1.33)
+    (fp_line (start -3.29 12.83) (end -3.29 -5.21)
       (stroke (width 0.12) (type solid)) (layer "F.SilkS"))
-    (fp_line (start 1.27 1.27) (end 1.27 -1.33)
+    (fp_line (start -1.98 -3.91) (end 4.52 -3.91)
       (stroke (width 0.12) (type solid)) (layer "F.SilkS"))
-    (fp_line (start 3.87 -1.33) (end 3.87 6.41)
+    (fp_line (start -1.98 1.76) (end -1.98 -3.91)
       (stroke (width 0.12) (type solid)) (layer "F.SilkS"))
-    (fp_line (start -1.8 -1.8) (end -1.8 6.85)
+    (fp_line (start -1.98 5.86) (end -3.29 5.86)
+      (stroke (width 0.12) (type solid)) (layer "F.SilkS"))
+    (fp_line (start -1.98 5.86) (end -1.98 5.86)
+      (stroke (width 0.12) (type solid)) (layer "F.SilkS"))
+    (fp_line (start -1.98 11.53) (end -1.98 5.86)
+      (stroke (width 0.12) (type solid)) (layer "F.SilkS"))
+    (fp_line (start 4.52 -3.91) (end 4.52 11.53)
+      (stroke (width 0.12) (type solid)) (layer "F.SilkS"))
+    (fp_line (start 4.52 11.53) (end -1.98 11.53)
+      (stroke (width 0.12) (type solid)) (layer "F.SilkS"))
+    (fp_line (start 5.83 -5.21) (end 5.83 12.83)
+      (stroke (width 0.12) (type solid)) (layer "F.SilkS"))
+    (fp_line (start 5.83 12.83) (end -3.29 12.83)
+      (stroke (width 0.12) (type solid)) (layer "F.SilkS"))
+    (fp_line (start -3.68 -5.6) (end -3.68 13.22)
       (stroke (width 0.05) (type solid)) (layer "F.CrtYd"))
-    (fp_line (start -1.8 6.85) (end 4.35 6.85)
+    (fp_line (start -3.68 13.22) (end 6.22 13.22)
       (stroke (width 0.05) (type solid)) (layer "F.CrtYd"))
-    (fp_line (start 4.35 -1.8) (end -1.8 -1.8)
+    (fp_line (start 6.22 -5.6) (end -3.68 -5.6)
       (stroke (width 0.05) (type solid)) (layer "F.CrtYd"))
-    (fp_line (start 4.35 6.85) (end 4.35 -1.8)
+    (fp_line (start 6.22 13.22) (end 6.22 -5.6)
       (stroke (width 0.05) (type solid)) (layer "F.CrtYd"))
-    (fp_line (start -1.27 0) (end 0 -1.27)
+    (fp_line (start -3.18 -4.1) (end -2.18 -5.1)
+      (stroke (width 0.1) (type solid)) (layer "F.Fab"))
+    (fp_line (start -3.18 1.76) (end -1.98 1.76)
+      (stroke (width 0.1) (type solid)) (layer "F.Fab"))
+    (fp_line (start -3.18 12.72) (end -3.18 -4.1)
+      (stroke (width 0.1) (type solid)) (layer "F.Fab"))
+    (fp_line (start -2.18 -5.1) (end 5.72 -5.1)
+      (stroke (width 0.1) (type solid)) (layer "F.Fab"))
+    (fp_line (start -1.98 -3.91) (end 4.52 -3.91)
+      (stroke (width 0.1) (type solid)) (layer "F.Fab"))
+    (fp_line (start -1.98 1.76) (end -1.98 -3.91)
+      (stroke (width 0.1) (type solid)) (layer "F.Fab"))
+    (fp_line (start -1.98 5.86) (end -3.18 5.86)
+      (stroke (width 0.1) (type solid)) (layer "F.Fab"))
+    (fp_line (start -1.98 5.86) (end -1.98 5.86)
+      (stroke (width 0.1) (type solid)) (layer "F.Fab"))
+    (fp_line (start -1.98 11.53) (end -1.98 5.86)
       (stroke (width 0.1) (type solid)) (layer "F.Fab"))
-    (fp_line (start -1.27 6.35) (end -1.27 0)
+    (fp_line (start 4.52 -3.91) (end 4.52 11.53)
       (stroke (width 0.1) (type solid)) (layer "F.Fab"))
-    (fp_line (start 0 -1.27) (end 3.81 -1.27)
+    (fp_line (start 4.52 11.53) (end -1.98 11.53)
       (stroke (width 0.1) (type solid)) (layer "F.Fab"))
-    (fp_line (start 3.81 -1.27) (end 3.81 6.35)
+    (fp_line (start 5.72 -5.1) (end 5.72 12.72)
       (stroke (width 0.1) (type solid)) (layer "F.Fab"))
-    (fp_line (start 3.81 6.35) (end -1.27 6.35)
+    (fp_line (start 5.72 12.72) (end -3.18 12.72)
       (stroke (width 0.1) (type solid)) (layer "F.Fab"))
-    (pad "1" thru_hole rect (at 0 0) (size 1.7 1.7) (drill 1) (layers "*.Cu" "*.Mask")
+    (pad "1" thru_hole roundrect (at 0 0) (size 1.7 1.7) (drill 1) (layers "*.Cu" "*.Mask") (roundrect_rratio 0.147059)
       (net 3 "GND") (pinfunction "Pin_1") (pintype "passive"))
-    (pad "2" thru_hole oval (at 2.54 0) (size 1.7 1.7) (drill 1) (layers "*.Cu" "*.Mask")
+    (pad "2" thru_hole circle (at 2.54 0) (size 1.7 1.7) (drill 1) (layers "*.Cu" "*.Mask")
       (net 18 "/Microcontrolador/SPI0_RX") (pinfunction "Pin_2") (pintype "passive"))
-    (pad "3" thru_hole oval (at 0 2.54) (size 1.7 1.7) (drill 1) (layers "*.Cu" "*.Mask")
+    (pad "3" thru_hole circle (at 0 2.54) (size 1.7 1.7) (drill 1) (layers "*.Cu" "*.Mask")
       (net 19 "/Microcontrolador/SPI0_CSn") (pinfunction "Pin_3") (pintype "passive"))
-    (pad "4" thru_hole oval (at 2.54 2.54) (size 1.7 1.7) (drill 1) (layers "*.Cu" "*.Mask")
+    (pad "4" thru_hole circle (at 2.54 2.54) (size 1.7 1.7) (drill 1) (layers "*.Cu" "*.Mask")
       (net 20 "/Microcontrolador/SPI0_SCK") (pinfunction "Pin_4") (pintype "passive"))
-    (pad "5" thru_hole oval (at 0 5.08) (size 1.7 1.7) (drill 1) (layers "*.Cu" "*.Mask")
+    (pad "5" thru_hole circle (at 0 5.08) (size 1.7 1.7) (drill 1) (layers "*.Cu" "*.Mask")
       (net 21 "/Microcontrolador/SPI0_TX") (pinfunction "Pin_5") (pintype "passive"))
-    (pad "6" thru_hole oval (at 2.54 5.08) (size 1.7 1.7) (drill 1) (layers "*.Cu" "*.Mask")
+    (pad "6" thru_hole circle (at 2.54 5.08) (size 1.7 1.7) (drill 1) (layers "*.Cu" "*.Mask")
       (net 52 "unconnected-(J3-Pin_6-Pad6)") (pinfunction "Pin_6") (pintype "passive+no_connect"))
-    (model "${KICAD6_3DMODEL_DIR}/Connector_PinHeader_2.54mm.3dshapes/PinHeader_2x03_P2.54mm_Vertical.wrl"
+    (pad "7" thru_hole circle (at 0 7.62) (size 1.7 1.7) (drill 1) (layers "*.Cu" "*.Mask"))
+    (pad "8" thru_hole circle (at 2.54 7.62) (size 1.7 1.7) (drill 1) (layers "*.Cu" "*.Mask"))
+    (model "${KICAD6_3DMODEL_DIR}/Connector_IDC.3dshapes/IDC-Header_2x04_P2.54mm_Vertical.wrl"
       (offset (xyz 0 0 0))
       (scale (xyz 1 1 1))
@@
     (fp_arc (start -1.11 49.69) (mid -1.433508 49.588809) (end -1.64 49.32)
       (stroke (width 0.12) (type solid)) (layer "F.SilkS"))
-    (fp_arc (start 18.89 -1.43) (mid 19.213529 -1.328823) (end 19.42 -1.06)
+    (fp_arc (start 18.89 -1.43) (mid 19.213491 -1.328806) (end 19.42 -1.06)
       (stroke (width 0.12) (type solid)) (layer "F.SilkS"))
-    (fp_arc (start 19.42 49.32) (mid 19.213497 49.588778) (end 18.89 49.69)
+    (fp_arc (start 19.42 49.32) (mid 19.213487 49.588772) (end 18.89 49.69)
       (stroke (width 0.12) (type solid)) (layer "F.SilkS"))
     (fp_poly
@@
   (segment (start 55.7615 101.6) (end 60.3335 106.172) (width 0.6) (layer "B.Cu") (net 20))
   (segment (start 52.07 101.6) (end 55.7615 101.6) (width 0.6) (layer "B.Cu") (net 20))
-  (segment (start 53.96 108.57) (end 66.1162 108.57) (width 0.6) (layer "B.Cu") (net 21))
-  (segment (start 49.53 104.14) (end 53.96 108.57) (width 0.6) (layer "B.Cu") (net 21))
+  (segment (start 48.18 105.49) (end 49.53 104.14) (width 0.6) (layer "B.Cu") (net 21))
+  (segment (start 66.1162 108.57) (end 49.510811 108.57) (width 0.6) (layer "B.Cu") (net 21))
+  (segment (start 48.18 107.239189) (end 48.18 105.49) (width 0.6) (layer "B.Cu") (net 21))
+  (segment (start 49.510811 108.57) (end 48.18 107.239189) (width 0.6) (layer "B.Cu") (net 21))
   (segment (start 45.6015 118.618) (end 60.5875 118.618) (width 0.6) (layer "F.Cu") (net 24))
   (segment (start 133.35 131.52) (end 133.35 130.21) (width 0.6) (layer "F.Cu") (net 24))

Commit message: ActualizaciónPCB_LogoUNCargador
Parts:
- added G***: LOGO, Logo_UNCargador:UNCargador_LogoGrande, B.Cu at (161.8, 43.8)
Routing:
- net GND: track 720.7 -> 722.6 mm
- net /Potencia2.0/N: track 53.9 -> 52.6 mm
- net +3.3V: track 303.3 -> 302.1 mm

Commit message: PCB_VersiónFinal_HD4K
Parts:
- added ?: , , F.Cu at (83.9, 139.0)
Routing:
- net GND: track 722.6 -> 0.00 mm, vias 30 -> 0
- net /Microcontrolador/TX_Pzem: track 209.1 -> 162.3 mm
- net Pilot_ADC: track 237.0 -> 199.5 mm
- net Net-(J5-Pin_3): track 34.3 -> 22.6 mm
- net +5V: track 294.6 -> 287.0 mm
- net /Microcontrolador/Pilot_PWM: track 192.6 -> 185.0 mm
- net Net-(C4-Pad1): track 53.2 -> 48.5 mm
- net +12V: track 280.0 -> 275.5 mm
- net /Microcontrolador/FALLA: track 95.4 -> 91.7 mm
- net Net-(U2--): track 40.7 -> 42.6 mm
- net Net-(D3-K): track 106.8 -> 105.6 mm
- net DisplaySDA: track 72.2 -> 71.6 mm
- net /Microcontrolador/GFCI_TEST: track 128.3 -> 127.7 mm

Commit message: PCB_Final
Parts:
- J3: footprint Connector_IDC:IDC-Header_2x04_P2.54mm_Vertical -> Connector_IDC:IDC-Header_2x05_P2.54mm_Vertical
Routing:
- net /Microcontrolador/SPI0_TX: track 22.1 -> 27.8 mm
Changed lines of the file:
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@@
     )
   )
-  (footprint "Connector_IDC:IDC-Header_2x04_P2.54mm_Vertical" (layer "F.Cu")
+  (footprint "Connector_IDC:IDC-Header_2x05_P2.54mm_Vertical" (layer "F.Cu")
     (at 49.53 99.06)
-    (descr "Through hole IDC box header, 2x04, 2.54mm pitch, DIN 41651 / IEC 60603-13, double rows, https://docs.google.com/spreadsheets/d/16SsEcesNF15N3Lb4niX7dcUr-NY5_MFPQhobNuNppn4/edit#gid=0")
-    (tags "Through hole vertical IDC box header THT 2x04 2.54mm double row")
+    (descr "Through hole IDC box header, 2x05, 2.54mm pitch, DIN 41651 / IEC 60603-13, double rows, https://docs.google.com/spreadsheets/d/16SsEcesNF15N3Lb4niX7dcUr-NY5_MFPQhobNuNppn4/edit#gid=0")
+    (tags "Through hole vertical IDC box header THT 2x05 2.54mm double row")
     (property "Sheetfile" "CircuitoPotencia.kicad_sch")
     (property "Sheetname" "")
@@
         (effects (font (size 1 1) (thickness 0.15)))
     )
-    (fp_text value "Conn_02x03_Counter_Clockwise" (at 1.27 13.72) (layer "F.Fab")
+    (fp_text value "Conn_02x03_Counter_Clockwise" (at 1.27 16.26) (layer "F.Fab")
         (effects (font (size 1 1) (thickness 0.15)))
     )
-    (fp_text user "${REFERENCE}" (at 1.27 3.81 90) (layer "F.Fab")
+    (fp_text user "${REFERENCE}" (at 1.27 5.08 90) (layer "F.Fab")
         (effects (font (size 1 1) (thickness 0.15)))
     )
@@
     (fp_line (start -3.29 -5.21) (end 5.83 -5.21)
       (stroke (width 0.12) (type solid)) (layer "F.SilkS"))
-    (fp_line (start -3.29 1.76) (end -1.98 1.76)
+    (fp_line (start -3.29 3.03) (end -1.98 3.03)
       (stroke (width 0.12) (type solid)) (layer "F.SilkS"))
-    (fp_line (start -3.29 12.83) (end -3.29 -5.21)
+    (fp_line (start -3.29 15.37) (end -3.29 -5.21)
       (stroke (width 0.12) (type solid)) (layer "F.SilkS"))
     (fp_line (start -1.98 -3.91) (end 4.52 -3.91)
       (stroke (width 0.12) (type solid)) (layer "F.SilkS"))
-    (fp_line (start -1.98 1.76) (end -1.98 -3.91)
+    (fp_line (start -1.98 3.03) (end -1.98 -3.91)
       (stroke (width 0.12) (type solid)) (layer "F.SilkS"))
-    (fp_line (start -1.98 5.86) (end -3.29 5.86)
+    (fp_line (start -1.98 7.13) (end -3.29 7.13)
       (stroke (width 0.12) (type solid)) (layer "F.SilkS"))
-    (fp_line (start -1.98 5.86) (end -1.98 5.86)
+    (fp_line (start -1.98 7.13) (end -1.98 7.13)
       (stroke (width 0.12) (type solid)) (layer "F.SilkS"))
-    (fp_line (start -1.98 11.53) (end -1.98 5.86)
+    (fp_line (start -1.98 14.07) (end -1.98 7.13)
       (stroke (width 0.12) (type solid)) (layer "F.SilkS"))
-    (fp_line (start 4.52 -3.91) (end 4.52 11.53)
+    (fp_line (start 4.52 -3.91) (end 4.52 14.07)
       (stroke (width 0.12) (type solid)) (layer "F.SilkS"))
-    (fp_line (start 4.52 11.53) (end -1.98 11.53)
+    (fp_line (start 4.52 14.07) (end -1.98 14.07)
       (stroke (width 0.12) (type solid)) (layer "F.SilkS"))
-    (fp_line (start 5.83 -5.21) (end 5.83 12.83)
+    (fp_line (start 5.83 -5.21) (end 5.83 15.37)
       (stroke (width 0.12) (type solid)) (layer "F.SilkS"))
-    (fp_line (start 5.83 12.83) (end -3.29 12.83)
+    (fp_line (start 5.83 15.37) (end -3.29 15.37)
       (stroke (width 0.12) (type solid)) (layer "F.SilkS"))
-    (fp_line (start -3.68 -5.6) (end -3.68 13.22)
+    (fp_line (start -3.68 -5.6) (end -3.68 15.76)
       (stroke (width 0.05) (type solid)) (layer "F.CrtYd"))
-    (fp_line (start -3.68 13.22) (end 6.22 13.22)
+    (fp_line (start -3.68 15.76) (end 6.22 15.76)
       (stroke (width 0.05) (type solid)) (layer "F.CrtYd"))
     (fp_line (start 6.22 -5.6) (end -3.68 -5.6)
       (stroke (width 0.05) (type solid)) (layer "F.CrtYd"))
-    (fp_line (start 6.22 13.22) (end 6.22 -5.6)
+    (fp_line (start 6.22 15.76) (end 6.22 -5.6)
       (stroke (width 0.05) (type solid)) (layer "F.CrtYd"))
     (fp_line (start -3.18 -4.1) (end -2.18 -5.1)
       (stroke (width 0.1) (type solid)) (layer "F.Fab"))
-    (fp_line (start -3.18 1.76) (end -1.98 1.76)
+    (fp_line (start -3.18 3.03) (end -1.98 3.03)
       (stroke (width 0.1) (type solid)) (layer "F.Fab"))
-    (fp_line (start -3.18 12.72) (end -3.18 -4.1)
+    (fp_line (start -3.18 15.26) (end -3.18 -4.1)
       (stroke (width 0.1) (type solid)) (layer "F.Fab"))
     (fp_line (start -2.18 -5.1) (end 5.72 -5.1)
@@
     (fp_line (start -1.98 -3.91) (end 4.52 -3.91)
       (stroke (width 0.1) (type solid)) (layer "F.Fab"))
-    (fp_line (start -1.98 1.76) (end -1.98 -3.91)
+    (fp_line (start -1.98 3.03) (end -1.98 -3.91)
       (stroke (width 0.1) (type solid)) (layer "F.Fab"))
-    (fp_line (start -1.98 5.86) (end -3.18 5.86)
+    (fp_line (start -1.98 7.13) (end -3.18 7.13)
       (stroke (width 0.1) (type solid)) (layer "F.Fab"))
-    (fp_line (start -1.98 5.86) (end -1.98 5.86)
+    (fp_line (start -1.98 7.13) (end -1.98 7.13)
       (stroke (width 0.1) (type solid)) (layer "F.Fab"))
-    (fp_line (start -1.98 11.53) (end -1.98 5.86)
+    (fp_line (start -1.98 14.07) (end -1.98 7.13)
       (stroke (width 0.1) (type solid)) (layer "F.Fab"))
-    (fp_line (start 4.52 -3.91) (end 4.52 11.53)
+    (fp_line (start 4.52 -3.91) (end 4.52 14.07)
       (stroke (width 0.1) (type solid)) (layer "F.Fab"))
-    (fp_line (start 4.52 11.53) (end -1.98 11.53)
+    (fp_line (start 4.52 14.07) (end -1.98 14.07)
       (stroke (width 0.1) (type solid)) (layer "F.Fab"))
-    (fp_line (start 5.72 -5.1) (end 5.72 12.72)
+    (fp_line (start 5.72 -5.1) (end 5.72 15.26)
       (stroke (width 0.1) (type solid)) (layer "F.Fab"))
-    (fp_line (start 5.72 12.72) (end -3.18 12.72)
+    (fp_line (start 5.72 15.26) (end -3.18 15.26)
       (stroke (width 0.1) (type solid)) (layer "F.Fab"))
     (pad "1" thru_hole roundrect (at 0 0) (size 1.7 1.7) (drill 1) (layers "*.Cu" "*.Mask") (roundrect_rratio 0.147059)
@@
     (pad "7" thru_hole circle (at 0 7.62) (size 1.7 1.7) (drill 1) (layers "*.Cu" "*.Mask"))
     (pad "8" thru_hole circle (at 2.54 7.62) (size 1.7 1.7) (drill 1) (layers "*.Cu" "*.Mask"))
-    (model "${KICAD6_3DMODEL_DIR}/Connector_IDC.3dshapes/IDC-Header_2x04_P2.54mm_Vertical.wrl"
+    (pad "9" thru_hole circle (at 0 10.16) (size 1.7 1.7) (drill 1) (layers "*.Cu" "*.Mask"))
+    (pad "10" thru_hole circle (at 2.54 10.16) (size 1.7 1.7) (drill 1) (layers "*.Cu" "*.Mask"))
+    (model "${KICAD6_3DMODEL_DIR}/Connector_IDC.3dshapes/IDC-Header_2x05_P2.54mm_Vertical.wrl"
       (offset (xyz 0 0 0))
       (scale (xyz 1 1 1))
@@
     (fp_arc (start -1.11 49.69) (mid -1.433508 49.588809) (end -1.64 49.32)
       (stroke (width 0.12) (type solid)) (layer "F.SilkS"))
-    (fp_arc (start 18.89 -1.43) (mid 19.213484 -1.328785) (end 19.42 -1.06)
+    (fp_arc (start 18.89 -1.43) (mid 19.213502 -1.328793) (end 19.42 -1.06)
       (stroke (width 0.12) (type solid)) (layer "F.SilkS"))
-    (fp_arc (start 19.42 49.32) (mid 19.213487 49.588772) (end 18.89 49.69)
+    (fp_arc (start 19.42 49.32) (mid 19.213496 49.58881) (end 18.89 49.69)
       (stroke (width 0.12) (type solid)) (layer "F.SilkS"))
     (fp_poly
@@
   (segment (start 52.07 101.6) (end 55.8292 101.6) (width 0.6) (layer "B.Cu") (net 20))
   (segment (start 55.8292 101.6) (end 60.2592 106.03) (width 0.6) (layer "B.Cu") (net 20))
-  (segment (start 48.18 105.49) (end 49.53 104.14) (width 0.6) (layer "B.Cu") (net 21))
-  (segment (start 66.1162 108.57) (end 49.510811 108.57) (width 0.6) (layer "B.Cu") (net 21))
-  (segment (start 48.18 107.239189) (end 48.18 105.49) (width 0.6) (layer "B.Cu") (net 21))
-  (segment (start 49.510811 108.57) (end 48.18 107.239189) (width 0.6) (layer "B.Cu") (net 21))
+  (segment (start 61.0362 111.1758) (end 48.6156 111.1758) (width 0.6) (layer "B.Cu") (net 21))
+  (segment (start 63.642 108.57) (end 61.0362 111.1758) (width 0.6) (layer "B.Cu") (net 21))
+  (segment (start 48.2092 104.14) (end 49.53 104.14) (width 0.6) (layer "B.Cu") (net 21))
+  (segment (start 66.1162 108.57) (end 63.642 108.57) (width 0.6) (layer "B.Cu") (net 21))
+  (segment (start 47.3964 104.9528) (end 48.2092 104.14) (width 0.6) (layer "B.Cu") (net 21))
+  (segment (start 47.3964 109.9566) (end 47.3964 104.9528) (width 0.6) (layer "B.Cu") (net 21))
+  (segment (start 48.6156 111.1758) (end 47.3964 109.9566) (width 0.6) (layer "B.Cu") (net 21))
   (segment (start 45.6015 118.618) (end 60.5875 118.618) (width 0.6) (layer "F.Cu") (net 24))
   (segment (start 133.35 131.52) (end 133.35 130.21) (width 0.6) (layer "F.Cu") (net 24))

Commit message: FinalPCB
Other:
- board size 143.9 x 141 mm -> 145 x 141 mm
